Commit message: first commit

File: rsc/camel_wire_arm/camel_wire_arm.urdf (robot description, URDF)
Before this commit: robot camel_wire_arm, 3 links, 2 joints
Links:
- link lower_arm: mass 10 -> 0.295
- link upper_arm: mass 0.7835 -> 0.295; geometry collision box size=0.2276 0.07775 0.090; visual mesh filename=fore_arm.stl scale=0.001 0.001 0.001
Joints:
- joint elbow_pitch: origin xyz=0 0.0 0.3345 rpy=0 0 0 -> xyz=0.2811 0 0.0474 rpy=1.570796 0 0

File: rsc/test_planar_elbow_2dof_point_mass.urdf (robot description, URDF)
Before this commit: robot test_planar_elbow_2dof, 7 links, 6 joints
Links:
- link point_mass_of_link1: mass 0.193 -> 0.3
- link point_mass_of_link2: mass 0.073 -> 0.05
